File: autonomous_control_board.kicad_pcb (KiCad board)
At the start: 2 copper layers, 72.1 x 60.1 mm, 9 parts, among them J1 Conn_01x15, J2 Conn_01x15, J3 Screw_Terminal_01x02, J4 Screw_Terminal_01x02, J5 Screw_Terminal_01x02, J6 Screw_Terminal_01x04, J7 Screw_Terminal_01x02, U1 L298N, U2 MCP4231-502E/P

Commit message: Small changes
Routing:
- net /CS: track 0.00 -> 16.2 mm
- net /GPIO23: track 20.6 -> 18.3 mm
- net /GPIO19: track 21.7 -> 19.5 mm
- net /GPIO18: track 10.9 -> 8.71 mm
Changed lines of the file:
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@@
 	)
 	(segment
-		(start 157.28 101.82)
-		(end 161.53 101.82)
+		(start 157.23 101.77)
+		(end 159.28 101.77)
 		(width 0.2)
 		(layer "B.Cu")
@@
 	(segment
 		(start 154.9 99.44)
-		(end 157.28 101.82)
+		(end 157.23 101.77)
 		(width 0.2)
 		(layer "B.Cu")
@@
 	)
 	(segment
-		(start 152.15 102.87)
-		(end 155.74 99.28)
+		(start 161.5 98)
+		(end 160.19 96.69)
+		(width 0.2)
+		(layer "F.Cu")
+		(net "/CS")
+	)
+	(segment
+		(start 160.19 96.69)
+		(end 159.28 96.69)
+		(width 0.2)
+		(layer "F.Cu")
+		(net "/CS")
+	)
+	(segment
+		(start 152.15 105.41)
+		(end 157.23 100.33)
+		(width 0.2)
+		(layer "F.Cu")
+		(net "/CS")
+	)
+	(segment
+		(start 157.23 100.33)
+		(end 160.92 100.33)
+		(width 0.2)
+		(layer "F.Cu")
+		(net "/CS")
+	)
+	(segment
+		(start 160.92 100.33)
+		(end 161.5 99.75)
+		(width 0.2)
+		(layer "F.Cu")
+		(net "/CS")
+	)
+	(segment
+		(start 161.5 99.75)
+		(end 161.5 98)
+		(width 0.2)
+		(layer "F.Cu")
+		(net "/CS")
+	)
+	(segment
+		(start 155.79 99.23)
+		(end 159.28 99.23)
 		(width 0.2)
 		(layer "F.Cu")
@@
 	)
 	(segment
-		(start 155.74 99.28)
-		(end 161.53 99.28)
+		(start 159.28 99.23)
+		(end 159.33 99.28)
 		(width 0.2)
 		(layer "F.Cu")
@@
 	)
 	(segment
-		(start 157.28 105.46)
-		(end 162.97 105.46)
+		(start 152.15 102.87)
+		(end 155.79 99.23)
+		(width 0.2)
+		(layer "F.Cu")
+		(net "/GPIO18")
+	)
+	(segment
+		(start 160.67 105.46)
+		(end 166.9 99.23)
 		(width 0.2)
 		(layer "B.Cu")
@@
 	)
 	(segment
-		(start 160.72 105.41)
-		(end 166.9 99.23)
+		(start 157.28 105.46)
+		(end 160.67 105.46)
 		(width 0.2)
 		(layer "B.Cu")
